Commit message: Removed automatic URDF import due to not beeing able to build it in VC; Tested System with gazebo UR5

File: Assets/Urdf/default/robot_description.urdf (robot description, URDF)
Before this commit: robot turtlebot, 35 links, 34 joints
Links:
- removed link base_footprint
- removed link camera_depth_frame
- removed link camera_depth_optical_frame
- removed link camera_link
- removed link camera_rgb_frame
- removed link camera_rgb_optical_frame
- removed link caster_back_link
- removed link caster_front_link
- removed link cliff_sensor_front_link
- removed link cliff_sensor_left_link
- removed link cliff_sensor_right_link
- removed link gyro_link
- removed link mount_asus_xtion_pro_link
- removed link plate_bottom_link
- removed link plate_middle_link
- removed link plate_top_link
- removed link pole_bottom_0_link
- removed link pole_bottom_1_link
- removed link pole_bottom_2_link
- removed link pole_bottom_3_link
- removed link pole_bottom_4_link
- removed link pole_bottom_5_link
- removed link pole_kinect_0_link
- removed link pole_kinect_1_link
- removed link pole_middle_0_link
- removed link pole_middle_1_link
- removed link pole_middle_2_link
- removed link pole_middle_3_link
- removed link pole_top_0_link
- removed link pole_top_1_link
- removed link pole_top_2_link
- removed link pole_top_3_link
- removed link wheel_left_link
- removed link wheel_right_link
- added link base
- added link ee_link; collision box size=0.01 0.01 0.01
- added link forearm_link, mass 2.275; collision mesh filename=package://ur_description/meshes/ur5/collision/forearm.stl; visual mesh filename=package://ur_description/meshes/ur5/visual/forearm.dae
- added link shoulder_link, mass 3.7; collision mesh filename=package://ur_description/meshes/ur5/collision/shoulder.stl; visual mesh filename=package://ur_description/meshes/ur5/visual/shoulder.dae
- added link tool0
- added link upper_arm_link, mass 8.393; collision mesh filename=package://ur_description/meshes/ur5/collision/upperarm.stl; visual mesh filename=package://ur_description/meshes/ur5/visual/upperarm.dae
- added link world
- added link wrist_1_link, mass 1.219; collision mesh filename=package://ur_description/meshes/ur5/collision/wrist1.stl; visual mesh filename=package://ur_description/meshes/ur5/visual/wrist1.dae
- added link wrist_2_link, mass 1.219; collision mesh filename=package://ur_description/meshes/ur5/collision/wrist2.stl; visual mesh filename=package://ur_description/meshes/ur5/visual/wrist2.dae
- added link wrist_3_link, mass 0.1879; collision mesh filename=package://ur_description/meshes/ur5/collision/wrist3.stl; visual mesh filename=package://ur_description/meshes/ur5/visual/wrist3.dae
- link base_link: mass 2.4 -> 4.0; geometry collision mesh filename=package://ur_description/meshes/ur5/collision/base.stl; visual mesh filename=package://ur_description/meshes/ur5/visual/base.dae
Joints:
- removed joint base_joint
- removed joint camera_depth_joint
- removed joint camera_depth_optical_joint
- removed joint camera_joint
- removed joint camera_rgb_joint
- removed joint camera_rgb_optical_joint
- removed joint caster_back_joint
- removed joint caster_front_joint
- removed joint cliff_sensor_front_joint
- removed joint cliff_sensor_left_joint
- removed joint cliff_sensor_right_joint
- removed joint gyro_joint
- removed joint mount_asus_xtion_pro_joint
- removed joint plate_bottom_joint
- removed joint plate_middle_joint
- removed joint plate_top_joint
- removed joint pole_bottom_0_joint
- removed joint pole_bottom_1_joint
- removed joint pole_bottom_2_joint
- removed joint pole_bottom_3_joint
- removed joint pole_bottom_4_joint
- removed joint pole_bottom_5_joint
- removed joint pole_kinect_0_joint
- removed joint pole_kinect_1_joint
- removed joint pole_middle_0_joint
- removed joint pole_middle_1_joint
- removed joint pole_middle_2_joint
- removed joint pole_middle_3_joint
- removed joint pole_top_0_joint
- removed joint pole_top_1_joint
- removed joint pole_top_2_joint
- removed joint pole_top_3_joint
- removed joint wheel_left_joint
- removed joint wheel_right_joint
- added joint base_link-base_fixed_joint: type fixed, parent base_link, child base, origin xyz=0 0 0 rpy=0 0 -3.14159265359
- added joint ee_fixed_joint: type fixed, parent wrist_3_link, child ee_link, origin xyz=0.0 0.0823 0.0 rpy=0.0 0.0 1.57079632679
- added joint elbow_joint: type revolute, parent upper_arm_link, child forearm_link, origin xyz=0.0 -0.1197 0.425 rpy=0.0 0.0 0.0, axis 0 1 0, limit lower=-3.14159265359 upper=3.14159265359 effort=150.0 velocity=3.15
- added joint shoulder_lift_joint: type revolute, parent shoulder_link, child upper_arm_link, origin xyz=0.0 0.13585 0.0 rpy=0.0 1.57079632679 0.0, axis 0 1 0, limit lower=-6.28318530718 upper=6.28318530718 effort=150.0 velocity=3.15
- added joint shoulder_pan_joint: type revolute, parent base_link, child shoulder_link, origin xyz=0.0 0.0 0.089159 rpy=0.0 0.0 0.0, axis 0 0 1, limit lower=-6.28318530718 upper=6.28318530718 effort=150.0 velocity=3.15
- added joint world_joint: type fixed, parent world, child base_link, origin xyz=0.0 0.0 0.0 rpy=0.0 0.0 0.0
- added joint wrist_1_joint: type revolute, parent forearm_link, child wrist_1_link, origin xyz=0.0 0.0 0.39225 rpy=0.0 1.57079632679 0.0, axis 0 1 0, limit lower=-6.28318530718 upper=6.28318530718 effort=28.0 velocity=3.2
- added joint wrist_2_joint: type revolute, parent wrist_1_link, child wrist_2_link, origin xyz=0.0 0.093 0.0 rpy=0.0 0.0 0.0, axis 0 0 1, limit lower=-6.28318530718 upper=6.28318530718 effort=28.0 velocity=3.2
- added joint wrist_3_joint: type revolute, parent wrist_2_link, child wrist_3_link, origin xyz=0.0 0.0 0.09465 rpy=0.0 0.0 0.0, axis 0 1 0, limit lower=-6.28318530718 upper=6.28318530718 effort=28.0 velocity=3.2
- added joint wrist_3_link-tool0_fixed_joint: type fixed, parent wrist_3_link, child tool0, origin xyz=0 0.0823 0 rpy=-1.57079632679 0 0
